File: HW/PawTrackWCH.kicad_sch (KiCad schematic)
At the start: 41 parts, among them J1 Batt_conn, J2 AUX_conn, J3 DBG_conn, P1 USB_C_Plug_USB2.0, Q1 AO3401A, SW1 User_btn, SW2 Reset_btn, U1 PJ4054B (LTC4054ES5), U2 CH582F, U3 BMI160/270/ICM42688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

Commit message: Use schottky instead of zener
Parts:
- removed D2: Zener, symbol Device:D_Zener_Small
- added D3: 1N5819WS, symbol Device:D_Schottky_Small
- Q1: value AO3401A -> CJ2305
Connections:
- net VBUS: now also D3.2 (A)
- net at C5.1, Q1.2 (S), U4.3 (VI): now also D3.1 (K)
Changed lines of the file:
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@@
       (effects (font (size 1.27 1.27)))
     )
-    (property "Value" "AO3401A" (at 106.68 39.37 90)
+    (property "Value" "CJ2305" (at 106.68 39.37 90)
       (effects (font (size 1.27 1.27)))
     )
@@
     )
   )
-  (symbol (lib_id "Device:D_Zener_Small") (at 113.03 50.8 180) (unit 1)
-    (in_bom yes) (on_board yes) (dnp no)
-    (property "Reference" "D2" (at 113.03 45.72 0)
-      (effects (font (size 1.27 1.27)))
-    )
-    (property "Value" "Zener" (at 113.03 48.26 0)
-      (effects (font (size 1.27 1.27)))
-    )
-    (property "Footprint" "" (at 113.03 50.8 90)
-      (effects (font (size 1.27 1.27)) hide)
-    )
-    (property "Datasheet" "~" (at 113.03 50.8 90)
-      (effects (font (size 1.27 1.27)) hide)
-    )
-    (pin "1")
-    (pin "2")
-    (instances
-      (project "PawTrackWCH"
-        (path "/1ef8389f-32dd-4802-ad62-64dcc44b8736"
-          (reference "D2") (unit 1)
-        )
-      )
-    )
-  )
   (symbol (lib_id "Device:Crystal_GND24") (at 95.25 133.35 90) (unit 1)
     (in_bom yes) (on_board yes) (dnp no)
@@
         )
       )
+    )
+  )
+  (symbol (lib_id "Device:D_Schottky_Small") (at 113.03 50.8 180) (unit 1)
+    (in_bom yes) (on_board yes) (dnp no)
+    (property "Reference" "D3" (at 113.03 45.72 0)
+      (effects (font (size 1.27 1.27)))
+    )
+    (property "Value" "1N5819WS" (at 113.03 48.26 0)
+      (effects (font (size 1.27 1.27)))
+    )
+    (property "Footprint" "" (at 113.03 50.8 90)
+      (effects (font (size 1.27 1.27)) hide)
+    )
+    (property "Datasheet" "~" (at 113.03 50.8 90)
+      (effects (font (size 1.27 1.27)) hide)
+    )
+    (pin "1")
+    (pin "2")
+    (instances
+      (project "PawTrackWCH"
+        (path "/1ef8389f-32dd-4802-ad62-64dcc44b8736"
+          (reference "D3") (unit 1)
+        )
+      )
